File: Schaltplan_box/Schaltplan_box.kicad_sch (KiCad schematic)
At the start: 10 parts, among them J1 6 Switches on top, J10 6 Switches on top, J11 Reset_mover, J2 Stepper_treiber_switcher, J3 Stepper_treiber_opener, J4 +VDC, J5 Reset_opener, J6 Mode_select, J9 Stepper_treiber_mover

Commit message: help
working mode 1 and kinda mode 0, not able to open box and not able to use mode 2
Parts:
- added J7: Reset_all, symbol Connector:Conn_01x02_Pin
Connections:
- net GND: now also J7.1 (Pin_1)
- net at A1.22 (A3): now also J7.2 (Pin_2)
Changed lines of the file:
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@@
+	(wire
+		(pts
+			(xy 161.29 76.2) (xy 144.78 76.2)
+		)
+		(stroke
+			(width 0)
+			(type default)
+		)
+	)
 	(wire
 		(pts
@@
 	(wire
 		(pts
+			(xy 144.78 76.2) (xy 144.78 88.9)
+		)
+		(stroke
+			(width 0)
+			(type default)
+		)
+	)
+	(wire
+		(pts
 			(xy 137.16 85.09) (xy 130.81 85.09)
 		)
@@
 	(wire
 		(pts
+			(xy 161.29 72.39) (xy 161.29 76.2)
+		)
+		(stroke
+			(width 0)
+			(type default)
+		)
+	)
+	(wire
+		(pts
 			(xy 193.04 121.92) (xy 193.04 140.97)
 		)
@@
 		(property "Intersheetrefs" "${INTERSHEET_REFS}"
 			(at 208.1809 143.51 0)
+			(effects
+				(font
+					(size 1.27 1.27)
+				)
+				(justify left)
+				(hide yes)
+			)
+		)
+	)
+	(global_label "GND"
+		(shape input)
+		(at 161.29 69.85 0)
+		(fields_autoplaced yes)
+		(effects
+			(font
+				(size 1.27 1.27)
+			)
+			(justify left)
+		)
+		(property "Intersheetrefs" "${INTERSHEET_REFS}"
+			(at 168.1457 69.85 0)
 			(effects
 				(font
@@
 					(unit 1)
 				)
+			)
+		)
+	)
+	(symbol
+		(lib_id "Connector:Conn_01x02_Pin")
+		(at 156.21 69.85 0)
+		(unit 1)
+		(exclude_from_sim no)
+		(in_bom yes)
+		(on_board yes)
+		(dnp no)
+		(property "Reference" "J7"
+			(at 156.845 64.77 0)
+			(effects
+				(font
+					(size 1.27 1.27)
+				)
+				(hide yes)
+			)
+		)
+		(property "Value" "Reset_all"
+			(at 159.258 58.674 90)
+			(effects
+				(font
+					(size 1.27 1.27)
+				)
+			)
+		)
+		(property "Footprint" ""
+			(at 156.21 69.85 0)
+			(effects
+				(font
+					(size 1.27 1.27)
+				)
+				(hide yes)
+			)
+		)
+		(property "Datasheet" "~"
+			(at 156.21 69.85 0)
+			(effects
+				(font
+					(size 1.27 1.27)
+				)
+				(hide yes)
+			)
+		)
+		(property "Description" "Generic connector, single row, 01x02, script generated"
+			(at 156.21 69.85 0)
+			(effects
+				(font
+					(size 1.27 1.27)
+				)
+				(hide yes)
+			)
+		)
+		(pin "1"
+		)
+		(pin "2"
+		)
+		(instances
+			(project "Schaltplan_box"
+				(path "/fda39497-1204-4cdb-bb61-daac59d8ab32"
+					(reference "J7")
+					(unit 1)
+				)
